Commit message: final project completed

File: src/my_robot_description/urdf/arm.xacro (robot description, xacro)
@@ -22,5 +22,5 @@
             <origin xyz="0 0 ${arm_base_height / 2.0}" rpy="0 0 0" />
         </collision>
-        <xacro:box_inertia m="5.0" x="${arm_base_length}" y="${arm_base_width}" z="${arm_base_height}"
+        <xacro:box_inertia m="0.5" x="${arm_base_length}" y="${arm_base_width}" z="${arm_base_height}"
             o_xyz="0 0 ${arm_base_height / 2.0}" o_rpy="0 0 0" />
     </link>

File: src/my_robot_description/urdf/my_robot.urdf.xacro (robot description, xacro)
@@ -4,4 +4,11 @@
     <xacro:include filename="mobile_base.xacro" />
     <xacro:include filename="mobile_base_gazebo.xacro" />
+    <xacro:include filename="arm.xacro" />
+    <xacro:include filename="arm_gazebo.xacro" />
     <xacro:include filename="camera.xacro" />
+    <joint name="mobile_base_arm_joint" type="fixed">
+        <parent link="base_link" />
+        <child link="arm_base_link" />
+        <origin xyz="${base_length / 4.0} 0 ${base_height}" rpy="0 0 0" />
+    </joint>
 </robot>
